Commit message: Update URDF files to reference new mesh filenames, modify collision parameters in process configurations, and enhance collision handling in inverse kinematics and rendering processes. Add gripper signal smoothing functionality and update data writing processes to include collision metrics.

File: assets/aloha_new_description/urdf/dual_piper.urdf (robot description, URDF)
Before this commit: robot dual_piper, 29 links, 28 joints
Links:
- link left_base_link: geometry collision mesh filename=package://aloha_new_description/meshes/base_link_col.STL; visual mesh filename=package://aloha_new_description/meshes/dark_dae/base_link.o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
- link left_link1: geometry collision mesh filename=package://aloha_new_description/meshes/link1_col.STL; visual mesh filename=package://aloha_new_description/meshes/dark_dae/link1.obj
- link left_link2: geometry collision mesh filename=package://aloha_new_description/meshes/link2_col.STL; visual mesh filename=package://aloha_new_description/meshes/dark_dae/link2.obj
- link left_link3: geometry collision mesh filename=package://aloha_new_description/meshes/link3_col.STL; visual mesh filename=package://aloha_new_description/meshes/dark_dae/link3.obj
- link left_link4: geometry collision mesh filename=package://aloha_new_description/meshes/link4_col.STL; visual mesh filename=package://aloha_new_description/meshes/dark_dae/link4.obj
- link left_link5: geometry collision mesh filename=package://aloha_new_description/meshes/link5_col.STL; visual mesh filename=package://aloha_new_description/meshes/dark_dae/link5.obj
- link right_base_link: geometry collision mesh filename=package://aloha_new_description/meshes/base_link_col.STL; visual mesh filename=package://aloha_new_description/meshes/dark_dae/base_link.o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
- link right_link1: geometry collision mesh filename=package://aloha_new_description/meshes/link1_col.STL; visual mesh filename=package://aloha_new_description/meshes/dark_dae/link1.obj
- link right_link2: geometry collision mesh filename=package://aloha_new_description/meshes/link2_col.STL; visual mesh filename=package://aloha_new_description/meshes/dark_dae/link2.obj
- link right_link3: geometry collision mesh filename=package://aloha_new_description/meshes/link3_col.STL; visual mesh filename=package://aloha_new_description/meshes/dark_dae/link3.obj
- link right_link4: geometry collision mesh filename=package://aloha_new_description/meshes/link4_col.STL; visual mesh filename=package://aloha_new_description/meshes/dark_dae/link4.obj
- link right_link5: geometry collision mesh filename=package://aloha_new_description/meshes/link5_col.STL; visual mesh filename=package://aloha_new_description/meshes/dark_dae/link5.obj

Commit message: Update dual_piper.urdf joint positions and disable render_filter in render.yaml
- Adjusted the `left_tcp_joint` and `right_tcp_joint` positions in `dual_piper.urdf` from 0.12 to 0.15 for improved alignment.
- Disabled the `render_filter` in `render.yaml` to modify rendering behavior.

File: assets/aloha_new_description/urdf/dual_piper.urdf (robot description, URDF)
Before this commit: robot dual_piper, 29 links, 28 joints
Joints:
- joint left_tcp_joint: origin xyz=0 0 0.12 rpy=0 0 0 -> xyz=0 0 0.15 rpy=0 0 0
- joint right_tcp_joint: origin xyz=0 0 0.12 rpy=0 0 0 -> xyz=0 0 0.15 rpy=0 0 0

Commit message: Update joint positions in dual_piper.urdf for improved alignment
- Adjusted the `left_tcp_joint` and `right_tcp_joint` positions from 0.15 to 0.14 to enhance the alignment of the robotic model.

File: assets/aloha_new_description/urdf/dual_piper.urdf (robot description, URDF)
Before this commit: robot dual_piper, 29 links, 28 joints
Joints:
- joint left_tcp_joint: origin xyz=0 0 0.15 rpy=0 0 0 -> xyz=0 0 0.14 rpy=0 0 0
- joint right_tcp_joint: origin xyz=0 0 0.15 rpy=0 0 0 -> xyz=0 0 0.14 rpy=0 0 0
